File: Mega68k.kicad_sch (KiCad schematic)
At the start: 16 parts, among them J1 CLK Select, J2 Ext CLK, J3 SPI, J4 Debug, SW1 ARD RESET, SW2 CPU_RESET, U1 68000D, X1 CXO_DIP8

Commit message: More tweaks to schematics before next rev V20220811
Parts:
- removed J1: CLK Select, Connector_PinHeader_2.54mm:PinHeader_1x03_P2.54mm_Vertical, symbol Connector:Conn_01x03_Male
- removed J2: Ext CLK, Connector_PinHeader_2.54mm:PinHeader_1x02_P2.54mm_Vertical, symbol Connector:Conn_01x02_Male
- removed J3: SPI, Connector_PinSocket_2.54mm:PinSocket_1x06_P2.54mm_Vertical, symbol Connector:Conn_01x06_Female
- removed U1: 68000D, Package_DIP:DIP-64_W22.86mm_Socket, symbol CPU_NXP_68000:68000D
- added C4, C5: 12pf, Capacitor_SMD:C_0603_1608Metric, symbol Device:C
- added C6: .1uF, Capacitor_SMD:C_0603_1608Metric, symbol Device:C
- added IC1: MC68008FN8, Package_LCC:PLCC-52_THT-Socket, symbol mc68k:MC68008FN8
- added J3: SD Card, Connector_PinSocket_2.54mm:PinSocket_1x08_P2.54mm_Vertical, symbol Connector:Conn_01x08_Female
- added J5: Serial 1, Connector_PinHeader_2.54mm:PinHeader_1x06_P2.54mm_Vertical, symbol Connector:Conn_01x06_Male
- added U1: AS6C4008-55PCN, Package_SO:SSOP-32_11.305x20.495mm_P1.27mm, symbol Memory_RAM:AS6C4008-55PCN
- added U2: MC68681FN, Package_LCC:PLCC-44_THT-Socket, symbol mc68k:MC68681FN
- added Y1: 3.6864, Crystal:Crystal_HC49-U_Vertical, symbol Device:Crystal
Connections:
- net ~{LDS} is gone; now on net ~{DS}: J4.46 (Pin_46)
- net A1: now also J4.4 (Pin_4), XA1.D48, IC1.52 (A1), U1.11 (A1), U2.4 (A2); no longer J4.3 (Pin_3), XA1.D49
- net A10: now also J4.13 (Pin_13), XA1.D35, IC1.9 (A10), U1.23 (A10); no longer J4.12 (Pin_12), XA1.D36
- net A11: now also J4.14 (Pin_14), XA1.D34, IC1.10 (A11), U1.25 (A11); no longer J4.13 (Pin_13), XA1.D35
- net A12: now also J4.15 (Pin_15), XA1.D33, IC1.11 (A12), U1.4 (A12); no longer J4.14 (Pin_14), XA1.D34
- net A13: now also J4.16 (Pin_16), XA1.D32, IC1.12 (A13), U1.28 (A13); no longer J4.15 (Pin_15), XA1.D33
- net A14: now also J4.17 (Pin_17), XA1.D31, IC1.14 (A14), U1.3 (A14); no longer J4.16 (Pin_16), XA1.D32
- net A15: now also J4.18 (Pin_18), XA1.D30, IC1.16 (A15), U1.31 (A15); no longer J4.17 (Pin_17), XA1.D31
- net A16: now also J4.19 (Pin_19), XA1.A0, IC1.18 (A16), U1.2 (A16); no longer J4.18 (Pin_18), XA1.D30
- net A17: now also J4.20 (Pin_20), XA1.A1, IC1.19 (A17), U1.30 (A17); no longer J4.19 (Pin_19), XA1.D53 (D53_SS)
- net A18: now also J4.21 (Pin_21), XA1.A2, IC1.20 (A18), U1.1 (A18); no longer J4.20 (Pin_20), XA1.D52
- net A19: now also J4.22 (Pin_22), XA1.A3, IC1.21 (A19); no longer J4.21 (Pin_21), XA1.D51
- net A2: now also J4.5 (Pin_5), XA1.D47, IC1.1 (A2), U1.10 (A2), U2.6 (A3); no longer J4.4 (Pin_4), XA1.D48
- net A20: now also J4.23 (Pin_23), XA1.A4, IC1.22 (A20); no longer J4.22 (Pin_22), XA1.D50
- net A21: now also J4.24 (Pin_24), XA1.A5, IC1.13 (A21); no longer J4.23 (Pin_23), XA1.D10
- net A3: now also J4.6 (Pin_6), XA1.D46, IC1.2 (A3), U1.9 (A3), U2.7 (A4); no longer J4.5 (Pin_5), XA1.D47
- net A4: now also J4.7 (Pin_7), XA1.D45, IC1.3 (A4), U1.8 (A4); no longer J4.6 (Pin_6), XA1.D46
- net A5: now also J4.8 (Pin_8), XA1.D44, IC1.4 (A5), U1.7 (A5); no longer J4.7 (Pin_7), XA1.D45
- net A6: now also J4.9 (Pin_9), XA1.D43, IC1.5 (A6), U1.6 (A6); no longer J4.8 (Pin_8), XA1.D44
- net A7: now also J4.10 (Pin_10), XA1.D42, IC1.6 (A7), U1.5 (A7); no longer J4.9 (Pin_9), XA1.D43
- net A8: now also J4.11 (Pin_11), XA1.D37, IC1.7 (A8), U1.27 (A8); no longer J4.10 (Pin_10), XA1.D42
- net A9: now also J4.12 (Pin_12), XA1.D36, IC1.8 (A9), U1.26 (A9); no longer J4.11 (Pin_11), XA1.D37
- net CPU_CLK: now also X1.5 (OUT), XA1.D9, IC1.38 (CLK)
- net D0: now also J4.27 (Pin_27), IC1.30 (D0), U1.13 (DQ0), U2.28 (D0); no longer J4.26 (Pin_26)
- net D1: now also J4.28 (Pin_28), IC1.29 (D1), U1.14 (DQ1), U2.18 (D1); no longer J4.27 (Pin_27)
- net D2: now also J4.29 (Pin_29), IC1.28 (D2), U1.15 (DQ2), U2.27 (D2); no longer J4.28 (Pin_28)
- net D3: now also J4.30 (Pin_30), IC1.27 (D3), U1.17 (DQ3), U2.19 (D3); no longer J4.29 (Pin_29)
- net D4: now also J4.31 (Pin_31), IC1.26 (D4), U1.18 (DQ4), U2.26 (D4); no longer J4.30 (Pin_30)
- net D5: now also J4.32 (Pin_32), IC1.25 (D5), U1.19 (DQ5), U2.20 (D5); no longer J4.31 (Pin_31)
- net D6: now also J4.33 (Pin_33), IC1.24 (D6), U1.20 (DQ6), U2.25 (D6); no longer J4.32 (Pin_32)
- net D7: now also J4.34 (Pin_34), IC1.23 (D7), U1.21 (DQ7), U2.21 (D7); no longer J4.33 (Pin_33)
- net E: now also XA1.A6, IC1.42 (E); no longer XA1.D13
- net FC0: now also XA1.A13, IC1.50 (FC0); no longer XA1.D17 (D17_RX2)
- net FC1: now also XA1.A14, IC1.49 (FC1); no longer XA1.D16 (D16_TX2)
- net FC2: now also XA1.A15, IC1.48 (FC2); no longer XA1.D6
- net GND: now also C4.1, C5.1, IC1.17 (GND_1), IC1.39 (GND_2), J3.6 (Pin_6), J5.6 (Pin_6), U1.16 (VSS), U2.22 (GND)
- net R~{W}: now also XA1.D8, IC1.33 (R/~{W}), U2.9 (R/~{W})
- net VCC: now also C6.1, IC1.15 (VCC), J3.8 (Pin_8), J5.4 (Pin_4), U1.32 (VCC), U2.44 (Vcc)
- net ~{AS}: now also XA1.D6, IC1.31 (~{AS})
- net ~{RAM_SEL}: now also XA1.D11, U1.22 (CE#); no longer XA1.D14 (D14_TX3)
- net ~{ROM_SEL}: no longer XA1.D15 (D15_RX3)
- net ~{OE}: now reaches J4.66 (Pin_66)
- net ~{OE}: now also XA1.D38, U1.24 (OE#)
- removed net A22: J4.24 (Pin_24), XA1.D11
- net A23: no longer names the net of J4.25 (Pin_25)
- net A23: no longer XA1.D12
- net AS: no longer names the net of XA1.D20 (D20_SDA)
- net BERR renamed ~{BERR}
- net ~{BERR}: now also IC1.44 (~{BERR})
- net BG renamed ~{BG}
- net ~{BG}: now also IC1.35 (~{BG})
- net BGACK renamed ~{BGACK}
- net ~{BGACK}: now also IC1.36 (~{BGACK})
- net BR renamed ~{BR}
- net ~{BR}: now also IC1.37 (~{BR})
- net D10: no longer names the net of J4.36 (Pin_36)
- net D10: no longer XA1.A2
- net D11: no longer names the net of J4.37 (Pin_37)
- net D11: no longer XA1.A3
- net D12: no longer names the net of J4.38 (Pin_38)
- net D12: no longer XA1.A4
- net D13: no longer names the net of J4.39 (Pin_39)
- net D13: no longer XA1.A5
- net D14: no longer names the net of J4.40 (Pin_40)
- net D14: no longer XA1.A6
- net D15: no longer names the net of XA1.A7
- net D15: no longer J4.41 (Pin_41)
- removed net D8: J4.34 (Pin_34), XA1.A0
- net D9: no longer names the net of J4.35 (Pin_35)
- net D9: no longer XA1.A1
- net DTACK renamed ~{DTACK}
- net ~{DTACK}: now also IC1.34 (~{DTACK})
- net HALT renamed ~{HALT}
- net ~{HALT}: now also IC1.40 (~{HALT})
- net INT_CLK: no longer names the net of XA1.D21 (D21_SCL)
- net INT_CLK: no longer X1.5 (OUT)
- net IPL0 renamed ~{IPL0}
- net ~{IPL0}: now also IC1.47 (~{IPL0})
- net IPL1 renamed ~{IPL1}
- net ~{IPL1}: now also IC1.45 (~{IPL1})
- net IPL2 renamed ~{IPL2}
- net ~{IPL2}: now also IC1.46 (~{IPL2}), U2.24 (~{INTRN})
- net LDS: no longer names the net of XA1.D19 (D19_RX1)
- net RESET renamed ~{RESET}
- net ~{RESET}: now also IC1.41 (~{RESET}), U2.38 (~{RESET})
- net R/W renamed ~{DS}
- net ~{DS}: now also IC1.32 (~{DS})
- net SPI_GND: no longer names the net of XA1.GND4 (SPI_GND)
- net SPI_MISO: no longer names the net of XA1.MOSI (SPI_MOSI)
- net SPI_MOSI: no longer names the net of XA1.MISO (SPI_MISO)
- net SPI_SCK: no longer names the net of XA1.SCK (SPI_SCK)
- net SPI_VCC: no longer names the net of XA1.5V2 (SPI_5V)
- net UDS: no longer names the net of XA1.D18 (D18_TX1)
- net VMA: no longer names the net of J4.52 (Pin_52)
- net VMA: no longer XA1.A13
- net VPA renamed ~{VPA}
- net ~{VPA}: now also IC1.43 (~{VPA})
- net ~{SDCARD_SEL} renamed ~{RAM_WE}
- net ~{RAM_WE}: now also XA1.D13, U1.29 (WE#); no longer XA1.D38
- net ~{UDS}: no longer names the net of J4.45 (Pin_45)
- new net 68681_X1: C4.2, U2.36 (X1/CLK), Y1.2
- new net 68681_X2: C5.2, U2.37 (X2), Y1.1
- new net A0: IC1.51 (A0), J4.3 (Pin_3), U1.12 (A0), U2.2 (A1), XA1.D49
- new net CTSA: J5.5 (Pin_5), U2.8 (IP0)
- new net CTSB: U2.5 (IP1)
- new net IP2: U2.40 (IP2)
- new net IP3: U2.3 (IP3)
- new net IP4: U2.43 (IP4)
- new net IP5: U2.42 (IP5)
- new net OP1: U2.14 (OP1)
- new net OP3: U2.15 (OP3)
- new net OP4: U2.30 (OP4)
- new net OP5: U2.16 (OP5)
- new net OP6: U2.29 (OP6)
- new net OP7: U2.17 (OP7)
- new net RTSA: J5.1 (Pin_1), U2.32 (OP0)
- new net RTSB: U2.31 (OP2)
- new net RxDA: J5.3 (Pin_3), U2.35 (RxDA)
- new net RxDB: U2.11 (RxDB)
- new net SDCLK: J3.5 (Pin_5), XA1.D52
- new net SDCS: J3.2 (Pin_2), XA1.D53 (D53_SS)
- new net SDD0: J3.4 (Pin_4), XA1.D50
- new net SDD1: J3.3 (Pin_3), XA1.D51
- new net TxDA: J5.2 (Pin_2), U2.33 (TxDA)
- new net TxDB: U2.13 (TxDB)
- new net ~{DTACK_UART}: U2.10 (~{DTACK}), XA1.D12
- new net ~{UART_SEL}: U2.39 (~{CS}), XA1.D10
- no-connect marks 15 -> 38
Other:
- note added: "UART CLK"
- moved on the sheet: C1, C2, D1, R1, XA1
