File: Mega68k.kicad_pcb (KiCad board)
At the start: 2 copper layers, 98.1 x 75.5 mm, 28 parts, among them J1 CLK Select, J2 Ext CLK, J3 SPI, J4 Debug, SW1 ARD RESET, SW2 CPU_RESET, U1 68000D, U4 74HC14, X1 CXO_DIP8

Commit message: More tweaks to schematics before next rev V20220811
Parts:
- removed D2: ROM, LED_SMD:LED_1206_3216Metric
- removed D3: RAM, LED_SMD:LED_1206_3216Metric
- removed D4: SD, LED_SMD:LED_1206_3216Metric
- removed D5: DTACK, LED_SMD:LED_1206_3216Metric
- removed J1: CLK Select, Connector_PinHeader_2.54mm:PinHeader_1x03_P2.54mm_Vertical
- removed J2: Ext CLK, Connector_PinHeader_2.54mm:PinHeader_1x02_P2.54mm_Vertical
- removed the J4 at (59.2, 118.6)
- removed R2, R3, R4, R5: 220, Resistor_SMD:R_0603_1608Metric
- removed REF**: KiCad-Logo2_8mm_SilkScreen, Symbol:KiCad-Logo2_8mm_SilkScreen
- removed U4: 74HC14, Package_SO:SOIC-14_3.9x8.7mm_P1.27mm
- added C4: 12pf, Capacitor_SMD:C_0603_1608Metric, F.Cu at (85.9, 71.5)
- added C5: 12pf, Capacitor_SMD:C_0603_1608Metric, F.Cu at (90.9, 71.5)
- added IC1: MC68008FN8, Package_LCC:PLCC-52_THT-Socket, F.Cu at (71.7, 81.9)
- added J5: Serial 1, Connector_PinHeader_2.54mm:PinHeader_1x06_P2.54mm_Vertical, F.Cu at (99.0, 65.2)
- added Logo1: KiCad-Logo2_8mm_SilkScreen, Symbol:KiCad-Logo2_8mm_SilkScreen, F.Cu at (128.5, 97.9)
- added Logo2: OSHW-Logo2_9.8x8mm_SilkScreen, Symbol:OSHW-Logo2_9.8x8mm_SilkScreen, F.Cu at (59.6, 69.1)
- added U2: MC68681FN, Package_LCC:PLCC-44_THT-Socket, F.Cu at (99.1, 80.0)
- added Y1: 3.6864, Crystal:Crystal_HC49-U_Vertical, F.Cu at (90.9, 66.5)
- C2: moved to F.Cu
- J3: value SPI -> SD Card; footprint Connector_PinSocket_2.54mm:PinSocket_1x06_P2.54mm_Vertical -> Connector_PinSocket_2.54mm:PinSocket_1x08_P2.54mm_Vertical
- U1: value 68000D -> AS6C4008-55PCN; footprint Package_DIP:DIP-64_W22.86mm_Socket -> Package_SO:SSOP-32_11.305x20.495mm_P1.27mm; moved to B.Cu
- moved J3 82.2 mm to (137.1, 76.7), turned to -90 degrees
- moved U1 68.7 mm to (128.3, 95.1), turned to 180 degrees
- moved SW1 51.7 mm to (131.2, 65.4)
- moved C2 41.4 mm to (56.8, 89.3), turned to -90 degrees
- moved R6 36.9 mm to (127.4, 65.4)
- moved SW2 36.8 mm to (117.0, 65.4)
- moved C7 33.0 mm to (128.3, 82.4)
- moved X1 31.3 mm to (71.2, 73.6)
- moved C3 30.6 mm to (66.8, 70.3)
- moved C6 27.8 mm to (102.5, 72.7), turned to 0 degrees
- moved D1 26.3 mm to (99.4, 103.5), turned to 0 degrees
- moved R1 21.6 mm to (104.9, 103.4), turned to 180 degrees
- moved C1 3.00 mm to (89.5, 103.5)
- moved J4 0.97 mm to (59.1, 53.2)
Connections:
- C6 pad 2: GND -> unconnected-(C6-Pad2)
- J3 pad 1: /SDCARD_SEL -> unconnected-(J3-Pad1)
- J3 pad 2: /SPI_SCK -> /SDCS
- J3 pad 3: /SPI_MOSI -> /SDD1
- J3 pad 4: /SPI_MISO -> /SDD0
- J3 pad 5: /SPI_VCC -> /SDCLK
- J3 pad 6: /SPI_GND -> GND
- J4 pad 10: /A8 -> /A7
- J4 pad 11: /A9 -> /A8
- J4 pad 12: /A10 -> /A9
- J4 pad 13: /A11 -> /A10
- J4 pad 14: /A12 -> /A11
- J4 pad 15: /A13 -> /A12
- J4 pad 16: /A14 -> /A13
- J4 pad 17: /A15 -> /A14
- J4 pad 18: /A16 -> /A15
- J4 pad 19: /A17 -> /A16
- J4 pad 20: /A18 -> /A17
- J4 pad 21: /A19 -> /A18
- J4 pad 22: /A20 -> /A19
- J4 pad 23: /A21 -> /A20
- J4 pad 24: /A22 -> /A21
- J4 pad 25: /A23 -> unconnected-(J4-Pad25)
- J4 pad 26: /D0 -> unconnected-(J4-Pad26)
- J4 pad 27: /D1 -> /D0
- J4 pad 28: /D2 -> /D1
- J4 pad 29: /D3 -> /D2
- J4 pad 3: /A1 -> /A0
- J4 pad 30: /D4 -> /D3
- J4 pad 31: /D5 -> /D4
- J4 pad 32: /D6 -> /D5
- J4 pad 33: /D7 -> /D6
- J4 pad 34: /D8 -> /D7
- J4 pad 35: /D9 -> unconnected-(J4-Pad35)
- J4 pad 36: /D10 -> unconnected-(J4-Pad36)
- J4 pad 37: /D11 -> unconnected-(J4-Pad37)
- J4 pad 38: /D12 -> unconnected-(J4-Pad38)
- J4 pad 39: /D13 -> unconnected-(J4-Pad39)
- J4 pad 4: /A2 -> /A1
- J4 pad 40: /D14 -> unconnected-(J4-Pad40)
- J4 pad 41: /D15 -> unconnected-(J4-Pad41)
- J4 pad 45: /~{UDS} -> unconnected-(J4-Pad45)
- J4 pad 46: /~{LDS} -> /~{DS}
- J4 pad 47: /RESET -> /~{RESET}
- J4 pad 48: /HALT -> /~{HALT}
- J4 pad 49: /BERR -> /~{BERR}
- J4 pad 5: /A3 -> /A2
- J4 pad 50: /DTACK -> /~{DTACK}
- J4 pad 52: /VMA -> unconnected-(J4-Pad52)
- J4 pad 53: /BGACK -> /~{BGACK}
- J4 pad 54: /VPA -> /~{VPA}
- J4 pad 55: /BR -> /~{BR}
- J4 pad 56: /BG -> /~{BG}
- J4 pad 57: /IPL0 -> /~{IPL0}
- J4 pad 58: /IPL1 -> /~{IPL1}
- J4 pad 59: /IPL2 -> /~{IPL2}
- J4 pad 6: /A4 -> /A3
- J4 pad 65: /~{SDCARD_SEL} -> /~{RAM_WE}
- J4 pad 66: unconnected-(J4-Pad66) -> /~{OE}
- J4 pad 7: /A5 -> /A4
- J4 pad 8: /A6 -> /A5
- J4 pad 9: /A7 -> /A6
- U1 pad 1: /D4 -> /A18
- U1 pad 10: /DTACK -> /A2
- U1 pad 11: /BG -> /A1
- U1 pad 12: /BGACK -> /A0
- U1 pad 13: /BR -> /D0
- U1 pad 14: VCC -> /D1
- U1 pad 15: /CPU_CLK -> /D2
- U1 pad 17: /HALT -> /D3
- U1 pad 18: /RESET -> /D4
- U1 pad 19: /VMA -> /D5
- U1 pad 2: /D3 -> /A16
- U1 pad 20: /E -> /D6
- U1 pad 21: /VPA -> /D7
- U1 pad 22: /BERR -> /~{RAM_SEL}
- U1 pad 23: /IPL2 -> /A10
- U1 pad 24: /IPL1 -> /~{OE}
- U1 pad 25: /IPL0 -> /A11
- U1 pad 26: /FC2 -> /A9
- U1 pad 27: /FC1 -> /A8
- U1 pad 28: /FC0 -> /A13
- U1 pad 29: /A1 -> /~{RAM_WE}
- U1 pad 3: /D2 -> /A14
- U1 pad 30: /A2 -> /A17
- U1 pad 31: /A3 -> /A15
- U1 pad 32: /A4 -> VCC
- U1 pad 4: /D1 -> /A12
- U1 pad 5: /D0 -> /A7
- U1 pad 6: /AS -> /A6
- U1 pad 7: /UDS -> /A5
- U1 pad 8: /LDS -> /A4
- U1 pad 9: /R/W -> /A3
- X1 pad 5: /INT_CLK -> /CPU_CLK
- XA1 pad 5V2: /SPI_VCC -> unconnected-(XA1-Pad5V2)
- XA1 pad A0: /D8 -> /A16
- XA1 pad A1: /D9 -> /A17
- XA1 pad A10: /BG -> /~{BG}
- XA1 pad A11: /BR -> /~{BR}
- XA1 pad A12: /VPA -> /~{VPA}
- XA1 pad A13: /VMA -> /FC0
- XA1 pad A14: unconnected-(XA1-PadA14) -> /FC1
- XA1 pad A15: unconnected-(XA1-PadA15) -> /FC2
- XA1 pad A2: /D10 -> /A18
- XA1 pad A3: /D11 -> /A19
- XA1 pad A4: /D12 -> /A20
- XA1 pad A5: /D13 -> /A21
- XA1 pad A6: /D14 -> /E
- XA1 pad A7: /D15 -> unconnected-(XA1-PadA7)
- XA1 pad A8: /BGACK -> /~{BGACK}
- XA1 pad A9: /BERR -> /~{BERR}
- XA1 pad D10: /A21 -> /~{UART_SEL}
- XA1 pad D11: /A22 -> /~{RAM_SEL}
- XA1 pad D12: /A23 -> /~{DTACK_UART}
- XA1 pad D13: /E -> /~{RAM_WE}
- XA1 pad D14: /~{RAM_SEL} -> unconnected-(XA1-PadD14)
- XA1 pad D15: /~{ROM_SEL} -> unconnected-(XA1-PadD15)
- XA1 pad D16: /FC1 -> unconnected-(XA1-PadD16)
- XA1 pad D17: /FC0 -> unconnected-(XA1-PadD17)
- XA1 pad D18: /UDS -> unconnected-(XA1-PadD18)
- XA1 pad D19: /LDS -> unconnected-(XA1-PadD19)
- XA1 pad D2: /IPL1 -> /~{IPL1}
- XA1 pad D20: /AS -> unconnected-(XA1-PadD20)
- XA1 pad D21: /INT_CLK -> unconnected-(XA1-PadD21)
- XA1 pad D3: /IPL0 -> /~{IPL0}
- XA1 pad D30: /A16 -> /A15
- XA1 pad D31: /A15 -> /A14
- XA1 pad D32: /A14 -> /A13
- XA1 pad D33: /A13 -> /A12
- XA1 pad D34: /A12 -> /A11
- XA1 pad D35: /A11 -> /A10
- XA1 pad D36: /A10 -> /A9
- XA1 pad D37: /A9 -> /A8
- XA1 pad D38: /~{SDCARD_SEL} -> /~{OE}
- XA1 pad D39: /DTACK -> /~{DTACK}
- XA1 pad D40: /RESET -> /~{RESET}
- XA1 pad D41: /HALT -> /~{HALT}
- XA1 pad D42: /A8 -> /A7
- XA1 pad D43: /A7 -> /A6
- XA1 pad D44: /A6 -> /A5
- XA1 pad D45: /A5 -> /A4
- XA1 pad D46: /A4 -> /A3
- XA1 pad D47: /A3 -> /A2
- XA1 pad D48: /A2 -> /A1
- XA1 pad D49: /A1 -> /A0
- XA1 pad D5: /IPL2 -> /~{IPL2}
- XA1 pad D50: /A20 -> /SDD0
- XA1 pad D51: /A19 -> /SDD1
- XA1 pad D52: /A18 -> /SDCLK
- XA1 pad D53: /A17 -> /SDCS
- XA1 pad D6: /FC2 -> /~{AS}
- XA1 pad D7: /R/W -> /~{DS}
- XA1 pad D8: unconnected-(XA1-PadD8) -> /R~{W}
- XA1 pad D9: unconnected-(XA1-PadD9) -> /CPU_CLK
- XA1 pad GND4: /SPI_GND -> unconnected-(XA1-PadGND4)
- XA1 pad MISO: /SPI_MOSI -> unconnected-(XA1-PadMISO)
- XA1 pad MOSI: /SPI_MISO -> unconnected-(XA1-PadMOSI)
- XA1 pad SCK: /SPI_SCK -> unconnected-(XA1-PadSCK)
Other:
- board size 98.1 x 75.5 mm -> 101.9 x 68.2 mm
- board text added: "CD"
- board text added: "CPU"
- board text added: "CS"
- board text added: "CTS"
- board text added: "D0"
- board text added: "D1"
- board text added: "RTS"
- board text added: "RX"
- board text added: "SD Card"
- board text added: "TX"
- board text added: "UART"
- board text added: "V20220811"
- board text added: "VCC"
- board text removed: "EXT"
- board text removed: "INT"
- board text removed: "v20220807"

Commit message: Added simple loop code and finalized board
Parts:
- J4: value Debug -> Bus
- moved Logo2 1.15 mm to (60.7, 69.5), turned to 90 degrees
Routing:
- net GND: track 0.00 -> 348.0 mm, vias 0 -> 3
- net /D0: track 0.00 -> 245.7 mm, vias 0 -> 2
- net VCC: track 0.00 -> 243.9 mm, vias 0 -> 1
- net /D5: track 0.00 -> 234.0 mm, vias 0 -> 2
- net /D7: track 0.00 -> 203.8 mm, vias 0 -> 4
- net /D1: track 0.00 -> 203.3 mm, vias 0 -> 3
- net /A13: track 0.00 -> 200.1 mm, vias 0 -> 2
- net /A6: track 0.00 -> 196.4 mm, vias 0 -> 1
- net /D3: track 0.00 -> 190.5 mm, vias 0 -> 3
- net /D4: track 0.00 -> 178.8 mm, vias 0 -> 3
- net /A8: track 0.00 -> 177.9 mm, vias 0 -> 1
- net /A5: track 0.00 -> 177.4 mm, vias 0 -> 2
- net /A11: track 0.00 -> 176.2 mm, vias 0 -> 2
- net /A7: track 0.00 -> 172.9 mm, vias 0 -> 2
- net /A15: track 0.00 -> 171.8 mm, vias 0 -> 3
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Other:
- board size 101.9 x 68.2 mm -> 101.8 x 68.2 mm
- board text added: "A0"
- board text added: "A1"
- board text added: "A10"
- board text added: "A11"
- board text added: "A12"
- board text added: "A13"
- board text added: "A14"
- board text added: "A15"
- board text added: "A16"
- board text added: "A17"
- board text added: "A18"
- board text added: "A19"
- board text added: "A2"
- board text added: "A20"
- board text added: "A21"
- board text added: "A3"
- board text added: "A4"
- board text added: "A5"
- board text added: "A6"
- board text added: "A7"
- board text added: "A8"
- board text added: "A9"
- board text added: "D3"
- board text added: "D4"
- board text added: "D5"
- board text added: "D6"
- board text added: "D7"
- board text added: "E"
- board text added: "R~{W}"
- board text added: "~{AS}"
- board text added: "~{BERR}"
- board text added: "~{BGACK}"
- board text added: "~{BG}"
- board text added: "~{BR}"
- board text added: "~{DS}"
- board text added: "~{DTACK}"
- board text added: "~{HALT}"
- board text added: "~{OE}"
- board text added: "~{RAMSL}"
- board text added: "~{RAMWE}"
- board text added: "~{RESET}"
- board text added: "~{ROMSL}"
- board text added: "~{VPA}"
