File: hardware/Mega68k.kicad_sch (KiCad schematic)
At the start: 21 parts, among them IC1 MC68008FN8, J3 SD Card, J4 Debug, J5 Serial 1, SW1 ARD RESET, SW2 CPU_RESET, U1 AS6C4008-55PCN, U2 MC68681FN, X1 CXO_DIP8, Y1 3.6864

Commit message: Some cleanup
Connections:
- net GND: now also C6.2
Changed lines of the file:
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@@
-    (stroke (width 0) (type default) (color 0 0 0 0))
-  )
-  (wire (pts (xy 213.995 66.04) (xy 213.995 55.88))
     (stroke (width 0) (type default) (color 0 0 0 0))
   )
@@
     (stroke (width 0) (type default) (color 0 0 0 0))
   )
-  (wire (pts (xy 213.995 73.66) (xy 213.995 77.47))
-    (stroke (width 0) (type default) (color 0 0 0 0))
-  )
   (wire (pts (xy 155.575 159.385) (xy 155.575 165.1))
     (stroke (width 0) (type default) (color 0 0 0 0))
@@
     (stroke (width 0) (type default) (color 0 0 0 0))
   )
+  (wire (pts (xy 213.995 55.88) (xy 213.995 77.47))
+    (stroke (width 0) (type default) (color 0 0 0 0))
+  )
